Commit message: try to add fetch_moveit_config

File: src/fetch_ros/fetch_description/robots/fetch.urdf (robot description, URDF)
Before this commit: robot fetch, 26 links, 25 joints
Links:
- added link l_back_support_wheel_link, mass 4.3542; collision mesh filename=package://fetch_description/meshes/l_wheel_link_collision.S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; visual mesh filename=package://fetch_description/meshes/l_wheel_link.STL
- added link l_front_support_wheel_link, mass 4.3542; collision mesh filename=package://fetch_description/meshes/l_wheel_link_collision.S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; visual mesh filename=package://fetch_description/meshes/l_wheel_link.STL
- added link r_back_support_wheel_link, mass 4.3542; collision mesh filename=package://fetch_description/meshes/r_wheel_link_collision.S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; visual mesh filename=package://fetch_description/meshes/r_wheel_link.STL
- added link r_front_support_wheel_link, mass 4.3542; collision mesh filename=package://fetch_description/meshes/r_wheel_link_collision.S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; visual mesh filename=package://fetch_description/meshes/r_wheel_link.STL
Joints:
- added joint l_back_support_wheel_joint: type continuous, parent base_link, child l_back_support_wheel_link, origin xyz=-0.21383 0.18738 0.055325 rpy=-6.123E-17 0 0, axis 0 1 0, limit effort=8.85 velocity=17.4
- added joint l_front_support_wheel_joint: type continuous, parent base_link, child l_front_support_wheel_link, origin xyz=0.21383 0.18738 0.055325 rpy=-6.123E-17 0 0, axis 0 1 0, limit effort=8.85 velocity=17.4
- added joint r_back_support_wheel_joint: type continuous, parent base_link, child r_back_support_wheel_link, origin xyz=-0.21383 -0.18738 0.055325 rpy=-6.123E-17 0 0, axis 0 1 0, limit effort=8.85 velocity=17.4
- added joint r_front_support_wheel_joint: type continuous, parent base_link, child r_front_support_wheel_link, origin xyz=0.21383 -0.18738 0.055325 rpy=-6.123E-17 0 0, axis 0 1 0, limit effort=8.85 velocity=17.4

Commit message: update robot infor for default state

File: src/fetch_ros/fetch_description/robots/fetch.urdf (robot description, URDF)
Before this commit: robot fetch, 30 links, 29 joints
Joints:
- joint bellows_joint: type fixed -> prismatic
